File: HW/HUB75-FPGA-Card/FTDI.kicad_sch (KiCad schematic)
At the start: 18 parts, among them U6 FT232H, U7 93LCxxBxxOT

Commit message: add usb audio implementation
Connections:
- net VIN renamed +5V
Changed lines of the file:
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@@
-    (stroke (width 0) (type default))
-  )
-  (wire (pts (xy 143.51 69.85) (xy 140.97 69.85))
     (stroke (width 0) (type default))
   )
@@
     (stroke (width 0) (type default))
   )
-  (wire (pts (xy 143.51 69.85) (xy 143.51 81.28))
+  (wire (pts (xy 143.51 78.74) (xy 143.51 81.28))
     (stroke (width 0) (type default))
   )
@@
     (effects (font (size 1.27 1.27)) (justify left))
   )
-  (hierarchical_label "VIN" (shape input) (at 140.97 69.85 180) (fields_autoplaced)
-    (effects (font (size 1.27 1.27)) (justify right))
-  )
   (hierarchical_label "D4" (shape output) (at 199.39 91.44 0) (fields_autoplaced)
     (effects (font (size 1.27 1.27)) (justify left))
   )
-  (hierarchical_label "USB_D+" (shape input) (at 148.59 99.06 180) (fields_autoplaced)
+  (hierarchical_label "USB_D+" (shape bidirectional) (at 148.59 99.06 180) (fields_autoplaced)
     (effects (font (size 1.27 1.27)) (justify right))
   )
@@
     (effects (font (size 1.27 1.27)) (justify left))
   )
-  (hierarchical_label "USB_D-" (shape input) (at 148.59 96.52 180) (fields_autoplaced)
+  (hierarchical_label "USB_D-" (shape bidirectional) (at 148.59 96.52 180) (fields_autoplaced)
     (effects (font (size 1.27 1.27)) (justify right))
   )
@@
         )
       )
+    )
+  )
+  (symbol (lib_id "power:+5V") (at 143.51 78.74 0) (unit 1)
+    (in_bom yes) (on_board yes) (dnp no) (fields_autoplaced)
+    (property "Reference" "#PWR064" (at 143.51 82.55 0)
+      (effects (font (size 1.27 1.27)) hide)
+    )
+    (property "Value" "+5V" (at 143.51 73.66 0)
+      (effects (font (size 1.27 1.27)))
+    )
+    (property "Footprint" "" (at 143.51 78.74 0)
+      (effects (font (size 1.27 1.27)) hide)
+    )
+    (property "Datasheet" "" (at 143.51 78.74 0)
+      (effects (font (size 1.27 1.27)) hide)
+    )
+    (pin "1")
+    (instances
+      (project "HUB75-FPGA-Card"
+        (path "/12c1dc17-a9d4-409d-a42e-fc131eeff0fd/befa8e28-726e-4ed7-b03c-a3e4bfcebff1"
+          (reference "#PWR064") (unit 1)
+        )
+        (path "/12c1dc17-a9d4-409d-a42e-fc131eeff0fd/a9a1e9cd-6574-4895-8694-62e6fb278fba"
+          (reference "#PWR039") (unit 1)
+        )
+      )

Commit message: finish up schematic and begin routing
Parts:
- removed FB1, FB2: FerriteBead, Resistor_SMD:R_0603_1608Metric_Pad0.98x0.95mm_HandSolder, symbol Device:FerriteBead
- added FB2, FB3: FerriteBead_Small, Resistor_SMD:R_0603_1608Metric, symbol Device:FerriteBead_Small
- C28: renamed from C10; footprint Capacitor_SMD:C_0603_1608Metric_Pad1.08x0.95mm_HandSolder -> Capacitor_SMD:C_0603_1608Metric
- C29: renamed from C11; footprint Capacitor_SMD:C_0603_1608Metric_Pad1.08x0.95mm_HandSolder -> Capacitor_SMD:C_0603_1608Metric
- C30: renamed from C12; footprint Capacitor_SMD:C_0603_1608Metric_Pad1.08x0.95mm_HandSolder -> Capacitor_SMD:C_0603_1608Metric
- C31: renamed from C13; footprint Capacitor_SMD:C_0603_1608Metric_Pad1.08x0.95mm_HandSolder -> Capacitor_SMD:C_0603_1608Metric
- C32: renamed from C14; footprint Capacitor_SMD:C_0603_1608Metric_Pad1.08x0.95mm_HandSolder -> Capacitor_SMD:C_0603_1608Metric
- C33: renamed from C6; footprint Capacitor_SMD:C_0603_1608Metric_Pad1.08x0.95mm_HandSolder -> Capacitor_SMD:C_0603_1608Metric
- C34: renamed from C8; footprint Capacitor_SMD:C_0603_1608Metric_Pad1.08x0.95mm_HandSolder -> Capacitor_SMD:C_0603_1608Metric
- C35: renamed from C5; footprint Capacitor_SMD:C_0603_1608Metric_Pad1.08x0.95mm_HandSolder -> Capacitor_SMD:C_0603_1608Metric
- R12: renamed from R15; footprint Resistor_SMD:R_0603_1608Metric_Pad0.98x0.95mm_HandSolder -> Resistor_SMD:R_0603_1608Metric
- R13: renamed from R11; footprint Resistor_SMD:R_0603_1608Metric_Pad0.98x0.95mm_HandSolder -> Resistor_SMD:R_0603_1608Metric
- R14: renamed from R12; footprint Resistor_SMD:R_0603_1608Metric_Pad0.98x0.95mm_HandSolder -> Resistor_SMD:R_0603_1608Metric
- R15: renamed from R14; footprint Resistor_SMD:R_0603_1608Metric_Pad0.98x0.95mm_HandSolder -> Resistor_SMD:R_0603_1608Metric
- R16: footprint Resistor_SMD:R_0603_1608Metric_Pad0.98x0.95mm_HandSolder -> Resistor_SMD:R_0603_1608Metric
- R17: renamed from R13; footprint Resistor_SMD:R_0603_1608Metric_Pad0.98x0.95mm_HandSolder -> Resistor_SMD:R_0603_1608Metric
- renumbered U6 to U7, U7 to U8
Connections:
- net +3.3VP: now also FB2.1, FB3.1
- net at C28.1, U7.3 (VPHY): now also FB2.2
- net at C29.1, U7.8 (VPLL): now also FB3.2
Other:
- note added: "EEPROM"
- moved on the sheet: C35, R13, R14, R15, R17, U8

Commit message: initial v1.1 board layout
still needs rp2040 pins routed
Parts:
- renumbered C35 to C27, C33 to C28, C34 to C29, C28 to C30, C29 to C31, C30 to C32, C31 to C33, C32 to C34, R13 to R12, R14 to R13, R17 to R14, R12 to R16, R16 to R17, U8 to U7, U7 to U8
Connections:
- net +5V is gone; now on net +3V3: U8.40 (VREGIN)
- net +3.3VP renamed +3V3
Other:
- note removed: "3.3VP is generated on VCCD by the 5V going to VREGIN and is only used by the FTDI/EEPROM"
