File: HW/Power-Module/Power-Module.kicad_pcb (KiCad board)
At the start: 2 copper layers, 42.4 x 29 mm, 26 parts, among them J1 USB_C_Receptacle_USB2.0_14P, J2 USB_C_Receptacle_USB2.0_14P, J3 USB_C_Receptacle_USB2.0_14P, J4 USB_C_Receptacle_USB2.0_14P, J5 Conn_01x02, U1 CH224K, U2 SY8366HQQC

Commit message: final v1.1 commit
boards ordered
Routing:
- net /USB_D-: track 34.2 -> 33.2 mm
- net GND: vias 10 -> 15
Changed lines of the file:
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@@
   (via (at 142.494 89.535) (size 0.8) (drill 0.4) (layers "F.Cu" "B.Cu") (free) (net 2))
   (via (at 154.559 93.152) (size 0.8) (drill 0.4) (layers "F.Cu" "B.Cu") (free) (net 2))
+  (via (at 148.082 96.52) (size 0.6) (drill 0.3) (layers "F.Cu" "B.Cu") (free) (net 2))
+  (via (at 142.494 101.6) (size 0.6) (drill 0.3) (layers "F.Cu" "B.Cu") (free) (net 2))
   (via (at 155.575 93.152) (size 0.8) (drill 0.4) (layers "F.Cu" "B.Cu") (free) (net 2))
   (via (at 145.669 98.679) (size 0.8) (drill 0.4) (layers "F.Cu" "B.Cu") (net 2))
   (via (at 145.542 89.535) (size 0.8) (drill 0.4) (layers "F.Cu" "B.Cu") (free) (net 2))
   (via (at 144.018 89.535) (size 0.8) (drill 0.4) (layers "F.Cu" "B.Cu") (free) (net 2))
+  (via (at 148.082 95.504) (size 0.6) (drill 0.3) (layers "F.Cu" "B.Cu") (free) (net 2))
   (via (at 147.066 89.535) (size 0.8) (drill 0.4) (layers "F.Cu" "B.Cu") (free) (net 2))
   (via (at 145.66157 97.814162) (size 0.8) (drill 0.4) (layers "F.Cu" "B.Cu") (net 2))
   (via (at 153.543 93.152) (size 0.8) (drill 0.4) (layers "F.Cu" "B.Cu") (free) (net 2))
   (via (at 156.591 93.152) (size 0.8) (drill 0.4) (layers "F.Cu" "B.Cu") (free) (net 2))
+  (via (at 148.336 94.234) (size 0.6) (drill 0.3) (layers "F.Cu" "B.Cu") (free) (net 2))
+  (via (at 142.494 93.472) (size 0.6) (drill 0.3) (layers "F.Cu" "B.Cu") (free) (net 2))
   (segment (start 136.938 101.552) (end 136.938 102.458) (width 0.25) (layer "F.Cu") (net 3))
   (segment (start 137.731 103.251) (end 139.179 103.251) (width 0.25) (layer "F.Cu") (net 3))
@@
   (segment (start 133.717059 98.36785) (end 133.709059 98.37585) (width 0.2413) (layer "F.Cu") (net 29))
   (segment (start 133.709059 98.37585) (end 133.640351 98.37585) (width 0.2413) (layer "F.Cu") (net 29))
-  (segment (start 133.640351 81.09585) (end 133.574501 81.03) (width 0.2413) (layer "F.Cu") (net 30))
   (segment (start 160.97265 80.777651) (end 160.97265 81.282349) (width 0.2413) (layer "F.Cu") (net 30))
-  (segment (start 159.287499 80.53) (end 159.221649 80.59585) (width 0.2413) (layer "F.Cu") (net 30))
-  (segment (start 135.807296 81.09585) (end 133.640351 81.09585) (width 0.2413) (layer "F.Cu") (net 30))
+  (segment (start 132.712 81.03) (end 133.6468 81.03) (width 0.2413) (layer "F.Cu") (net 30))
   (segment (start 131.838 82.03) (end 131.572 82.296) (width 0.2413) (layer "F.Cu") (net 30))
-  (segment (start 136.307296 80.59585) (end 135.807296 81.09585) (width 0.2413) (layer "F.Cu") (net 30))
-  (segment (start 133.574501 81.03) (end 132.712 81.03) (width 0.2413) (layer "F.Cu") (net 30))
-  (segment (start 159.221649 80.59585) (end 136.307296 80.59585) (width 0.2413) (layer "F.Cu") (net 30))
+  (segment (start 158.75 80.8188) (end 133.858 80.8188) (width 0.77) (layer "F.Cu") (net 30))
+  (segment (start 159.312146 80.772) (end 158.7968 80.772) (width 0.2413) (layer "F.Cu") (net 30))
   (segment (start 160.97265 81.282349) (end 160.724999 81.53) (width 0.2413) (layer "F.Cu") (net 30))
-  (segment (start 160.15 80.53) (end 159.287499 80.53) (width 0.2413) (layer "F.Cu") (net 30))
+  (segment (start 133.6468 81.03) (end 133.858 80.8188) (width 0.2413) (layer "F.Cu") (net 30))
+  (segment (start 160.15 80.53) (end 159.554146 80.53) (width 0.2413) (layer "F.Cu") (net 30))
   (segment (start 160.724999 81.53) (end 160.15 81.53) (width 0.2413) (layer "F.Cu") (net 30))
   (segment (start 160.724999 80.53) (end 160.97265 80.777651) (width 0.2413) (layer "F.Cu") (net 30))
   (segment (start 132.712 81.03) (end 131.576 81.03) (width 0.2413) (layer "F.Cu") (net 30))
   (segment (start 132.712 82.03) (end 131.838 82.03) (width 0.2413) (layer "F.Cu") (net 30))
+  (segment (start 158.7968 80.772) (end 158.75 80.8188) (width 0.2413) (layer "F.Cu") (net 30))
   (segment (start 160.15 80.53) (end 160.724999 80.53) (width 0.2413) (layer "F.Cu") (net 30))
   (segment (start 131.576 81.03) (end 131.572 81.026) (width 0.2413) (layer "F.Cu") (net 30))
+  (segment (start 159.554146 80.53) (end 159.312146 80.772) (width 0.2413) (layer "F.Cu") (net 30))
   (via (at 131.572 82.296) (size 0.6) (drill 0.3) (layers "F.Cu" "B.Cu") (net 30))
   (via (at 131.572 81.026) (size 0.6) (drill 0.3) (layers "F.Cu" "B.Cu") (net 30))
   (segment (start 131.572 82.296) (end 131.572 81.026) (width 0.2413) (layer "B.Cu") (net 30))
-  (segment (start 159.287499 81.03) (end 159.221649 80.96415) (width 0.2413) (layer "F.Cu") (net 31))
+  (segment (start 159.32735 81.319276) (end 159.32735 81.782349) (width 0.2413) (layer "F.Cu") (net 31))
+  (segment (start 160.15 81.03) (end 159.616626 81.03) (width 0.2413) (layer "F.Cu") (net 31))
+  (segment (start 159.32735 81.782349) (end 159.286201 81.7412) (width 0.2413) (layer "F.Cu") (net 31))
   (segment (start 131.02435 80.799155) (end 131.345155 80.47835) (width 0.2413) (layer "F.Cu") (net 31))
-  (segment (start 133.574501 81.53) (end 132.712 81.53) (width 0.2413) (layer "F.Cu") (net 31))
+  (segment (start 133.6468 81.53) (end 133.858 81.7412) (width 0.2413) (layer "F.Cu") (net 31))
+  (segment (start 159.286201 81.7412) (end 158.75 81.7412) (width 0.2413) (layer "F.Cu") (net 31))
   (segment (start 132.712 81.53) (end 132.66835 81.57365) (width 0.2413) (layer "F.Cu") (net 31))
   (segment (start 131.345155 80.47835) (end 132.66035 80.47835) (width 0.2413) (layer "F.Cu") (net 31))
-  (segment (start 159.221649 80.96415) (end 136.45985 80.96415) (width 0.2413) (layer "F.Cu") (net 31))
   (segment (start 159.575001 82.03) (end 160.15 82.03) (width 0.2413) (layer "F.Cu") (net 31))
   (segment (start 132.66035 80.47835) (end 132.712 80.53) (width 0.2413) (layer "F.Cu") (net 31))
   (segment (start 159.32735 81.782349) (end 159.575001 82.03) (width 0.2413) (layer "F.Cu") (net 31))
   (segment (start 131.345155 81.57365) (end 131.02435 81.252845) (width 0.2413) (layer "F.Cu") (net 31))
-  (segment (start 159.575001 81.03) (end 159.32735 81.277651) (width 0.2413) (layer "F.Cu") (net 31))
-  (segment (start 133.640351 81.46415) (end 133.574501 81.53) (width 0.2413) (layer "F.Cu") (net 31))
+  (segment (start 158.75 81.7412) (end 133.858 81.7412) (width 0.77) (layer "F.Cu") (net 31))
+  (segment (start 159.616626 81.03) (end 159.32735 81.319276) (width 0.2413) (layer "F.Cu") (net 31))
+  (segment (start 132.712 81.53) (end 133.6468 81.53) (width 0.2413) (layer "F.Cu") (net 31))
   (segment (start 131.02435 81.252845) (end 131.02435 80.799155) (width 0.2413) (layer "F.Cu") (net 31))
   (segment (start 132.66835 81.57365) (end 131.345155 81.57365) (width 0.2413) (layer "F.Cu") (net 31))
-  (segment (start 135.95985 81.46415) (end 133.640351 81.46415) (width 0.2413) (layer "F.Cu") (net 31))
-  (segment (start 159.32735 81.277651) (end 159.32735 81.782349) (width 0.2413) (layer "F.Cu") (net 31))
-  (segment (start 136.45985 80.96415) (end 135.95985 81.46415) (width 0.2413) (layer "F.Cu") (net 31))
-  (segment (start 160.15 81.03) (end 159.575001 81.03) (width 0.2413) (layer "F.Cu") (net 31))
-  (segment (start 160.15 81.03) (end 159.287499 81.03) (width 0.2413) (layer "F.Cu") (net 31))
   (zone (net 25) (net_name "/Buck/LX") (layer "F.Cu") (hatch edge 0.5)
     (priority 2)
@@
         (xy 151.257 102.743)
         (xy 151.257 97.155)
-        (xy 147.955 97.155)
-        (xy 147.955 95.504)
+        (xy 148.717 97.155)
+        (xy 148.717 95.504)
         (xy 156.591 95.504)
         (xy 156.591 102.743)
