File: HW/Power-Module/Power-Module.kicad_sch (KiCad schematic)
At the start: 13 parts, among them J1 USB_C_Receptacle_USB2.0_14P, J2 USB_C_Receptacle_USB2.0_14P, J3 USB_C_Receptacle_USB2.0_14P, J4 USB_C_Receptacle_USB2.0_14P, J5 Conn_01x02, U1 CH224K

Commit message: migrate to kicad 8
Parts:
- H1, H2, JP1: now left out of the parts list
